Commit message: Improve Gazebo simulation: park world, proper drone, moving person
World: Replace empty gray scene with a park environment — blue sky with
clouds, 9 trees (oak + pine from Gazebo model DB), two benches, a
concrete footpath, and a Gazebo actor (walk.dae) that walks a 44-second
rectangular patrol path instead of the previous static person_standing model.

Drone: Replace flat box with a proper quadrotor silhouette — small central
hub (0.18×0.18×0.06 m) plus four arms in X-configuration and four rotor
discs at the arm tips. Physics collision box and all sensor plugins are
unchanged.

Launch: Remove the redundant person_standing spawn node; the walking actor
is now embedded in the world file.

File: interceptor_ws/src/interceptor_drone/urdf/interceptor_quadrotor.urdf.xacro (robot description, xacro)
@@ -7,5 +7,68 @@
   <xacro:property name="camera_height" value="0.04"/>
   <xacro:property name="camera_depth" value="0.03"/>
-  <!-- Base link (simplified quadrotor) -->
+  <xacro:property name="arm_length" value="0.28"/>
+  <!--
+    Arm macro: thin box extending arm_length along the local +X axis.
+    Joint rotation (yaw) orients the arm in the X-config layout.
+  -->
+  <xacro:macro name="quad_arm" params="name yaw">
+    <link name="arm_${name}">
+      <inertial>
+        <mass value="0.025"/>
+        <inertia ixx="1e-5" ixy="0" ixz="0" iyy="1e-5" iyz="0" izz="1e-5"/>
+      </inertial>
+      <visual>
+        <origin xyz="${arm_length/2} 0 0" rpy="0 0 0"/>
+        <geometry>
+          <box size="${arm_length} 0.022 0.022"/>
+        </geometry>
+        <material name="arm_dark">
+          <color rgba="0.18 0.18 0.18 1"/>
+        </material>
+      </visual>
+    </link>
+    <joint name="arm_${name}_joint" type="fixed">
+      <parent link="base_link"/>
+      <child link="arm_${name}"/>
+      <origin xyz="0 0 0" rpy="0 0 ${yaw}"/>
+    </joint>
+  </xacro:macro>
+  <!-- X-configuration: FR=-45°, FL=+45°, RL=+135°, RR=-135° -->
+  <xacro:quad_arm name="fr" yaw="${-pi/4}"/>
+  <xacro:quad_arm name="fl" yaw="${pi/4}"/>
+  <xacro:quad_arm name="rl" yaw="${3*pi/4}"/>
+  <xacro:quad_arm name="rr" yaw="${-3*pi/4}"/>
+  <!--
+    Rotor macro: flat disc cylinder above the arm tip.
+    x/y are the arm tip positions in base_link frame (arm_length * cos/sin(45°) = 0.198).
+  -->
+  <xacro:macro name="quad_rotor" params="name x y">
+    <link name="rotor_${name}">
+      <inertial>
+        <mass value="0.01"/>
+        <inertia ixx="1e-5" ixy="0" ixz="0" iyy="1e-5" iyz="0" izz="1e-5"/>
+      </inertial>
+      <visual>
+        <origin xyz="0 0 0" rpy="0 0 0"/>
+        <geometry>
+          <cylinder radius="0.12" length="0.005"/>
+        </geometry>
+        <material name="rotor_gray">
+          <color rgba="0.6 0.6 0.6 0.85"/>
+        </material>
+      </visual>
+    </link>
+    <joint name="rotor_${name}_joint" type="fixed">
+      <parent link="base_link"/>
+      <child link="rotor_${name}"/>
+      <origin xyz="${x} ${y} 0.03" rpy="0 0 0"/>
+    </joint>
+  </xacro:macro>
+  <!-- arm_length * cos(45°) = 0.28 * 0.7071 = 0.198 -->
+  <xacro:quad_rotor name="fr" x=" 0.198" y="-0.198"/>
+  <xacro:quad_rotor name="fl" x=" 0.198" y=" 0.198"/>
+  <xacro:quad_rotor name="rl" x="-0.198" y=" 0.198"/>
+  <xacro:quad_rotor name="rr" x="-0.198" y="-0.198"/>
+  <!-- Base link: central hub (inertia and collision unchanged for physics) -->
   <link name="base_link">
     <inertial>
@@ -14,12 +77,14 @@
     </inertial>
     <visual>
-      <geometry>
-        <box size="0.4 0.4 0.1"/>
-      </geometry>
-      <material name="black">
-        <color rgba="0.1 0.1 0.1 1"/>
+      <!-- Small central hub — arms provide the full quad silhouette -->
+      <geometry>
+        <box size="0.18 0.18 0.06"/>
+      </geometry>
+      <material name="body_dark">
+        <color rgba="0.12 0.12 0.12 1"/>
       </material>
     </visual>
     <collision>
+      <!-- Keep original bounding box for physics accuracy -->
       <geometry>
         <box size="0.4 0.4 0.1"/>
@@ -79,5 +144,5 @@
     <origin xyz="0 ${baseline/2} 0" rpy="0 0 0"/>
   </joint>
-  <!-- Left camera optical link (for ROS conventions) -->
+  <!-- Left camera optical link (ROS convention: Z forward, X right, Y down) -->
   <link name="stereo_left_camera_optical_frame"/>
   <joint name="stereo_left_camera_optical_joint" type="fixed">
