Commit message: Replace box drone with realistic Holybro X500 V2 model
Swap the box/disc placeholder visuals for the PX4 x500 meshes
(PX4/PX4-gazebo-models, BSD-3-Clause): textured carbon-fibre frame,
5010 motors and 11" props, plus a ZED-class stereo housing.

- Frame mesh reduced from 22 MB to 8 MB with scripts/reduce_x500_mesh.py
  (only untextured parts decimated, carbon fibre kept at full detail).
- Mass, inertia, main collision box, IMU and stereo baseline unchanged;
  landing-gear collisions added so the drone rests on its skids.
- Stereo camera moved from the top plate (inside the prop discs) to
  under the payload rails: mount z 0.05 -> -0.0375 m, still published
  through TF from the URDF.
- Meshes installed and exported via gazebo_model_path so
  package:// URIs resolve in Gazebo Classic.

Co-Authored-By: Claude Opus 5.5 <noreply@anthropic.com>
Claude-Session: https://claude.ai/code/session_011dzjWSXGEFp5yaJJCdCJYz

File: interceptor_ws/src/interceptor_drone/urdf/interceptor_quadrotor.urdf.xacro (robot description, xacro)
@@ -1,74 +1,23 @@
 <?xml version="1.0"?>
 <robot xmlns:xacro="http://www.ros.org/wiki/xacro" name="interceptor_quadrotor">
+  <!--
+    Visual model: Holybro X500 V2 quadrotor (500 mm wheelbase, carbon-fibre
+    frame), meshes from PX4-gazebo-models (BSD-3-Clause), see meshes/x500/README.md.
+    Inertia, total mass, main collision box, IMU and the stereo baseline are
+    unchanged. Landing-gear collisions let the drone rest on its skids, and the
+    stereo camera hangs under the payload rails so it clears the propellers.
+  -->
   <!-- Property definitions -->
+  <xacro:property name="mesh_dir" value="package://interceptor_drone/meshes/x500"/>
   <xacro:property name="camera_mass" value="0.1"/>
   <xacro:property name="baseline" value="0.12"/>
-  <xacro:property name="camera_width" value="0.1"/>
-  <xacro:property name="camera_height" value="0.04"/>
-  <xacro:property name="camera_depth" value="0.03"/>
-  <xacro:property name="arm_length" value="0.28"/>
-  <!--
-    Arm macro: thin box extending arm_length along the local +X axis.
-    Joint rotation (yaw) orients the arm in the X-config layout.
-  -->
-  <xacro:macro name="quad_arm" params="name yaw">
-    <link name="arm_${name}">
-      <inertial>
-        <mass value="0.025"/>
-        <inertia ixx="1e-5" ixy="0" ixz="0" iyy="1e-5" iyz="0" izz="1e-5"/>
-      </inertial>
-      <visual>
-        <origin xyz="${arm_length/2} 0 0" rpy="0 0 0"/>
-        <geometry>
-          <box size="${arm_length} 0.022 0.022"/>
-        </geometry>
-        <material name="arm_dark">
-          <color rgba="0.18 0.18 0.18 1"/>
-        </material>
-      </visual>
-    </link>
-    <joint name="arm_${name}_joint" type="fixed">
-      <parent link="base_link"/>
-      <child link="arm_${name}"/>
-      <origin xyz="0 0 0" rpy="0 0 ${yaw}"/>
-    </joint>
-  </xacro:macro>
-  <!-- X-configuration: FR=-45°, FL=+45°, RL=+135°, RR=-135° -->
-  <xacro:quad_arm name="fr" yaw="${-pi/4}"/>
-  <xacro:quad_arm name="fl" yaw="${pi/4}"/>
-  <xacro:quad_arm name="rl" yaw="${3*pi/4}"/>
-  <xacro:quad_arm name="rr" yaw="${-3*pi/4}"/>
-  <!--
-    Rotor macro: flat disc cylinder above the arm tip.
-    x/y are the arm tip positions in base_link frame (arm_length * cos/sin(45°) = 0.198).
-  -->
-  <xacro:macro name="quad_rotor" params="name x y">
-    <link name="rotor_${name}">
-      <inertial>
-        <mass value="0.01"/>
-        <inertia ixx="1e-5" ixy="0" ixz="0" iyy="1e-5" iyz="0" izz="1e-5"/>
-      </inertial>
-      <visual>
-        <origin xyz="0 0 0" rpy="0 0 0"/>
-        <geometry>
-          <cylinder radius="0.12" length="0.005"/>
-        </geometry>
-        <material name="rotor_gray">
-          <color rgba="0.6 0.6 0.6 0.85"/>
-        </material>
-      </visual>
-    </link>
-    <joint name="rotor_${name}_joint" type="fixed">
-      <parent link="base_link"/>
-      <child link="rotor_${name}"/>
-      <origin xyz="${x} ${y} 0.03" rpy="0 0 0"/>
-    </joint>
-  </xacro:macro>
-  <!-- arm_length * cos(45°) = 0.28 * 0.7071 = 0.198 -->
-  <xacro:quad_rotor name="fr" x=" 0.198" y="-0.198"/>
-  <xacro:quad_rotor name="fl" x=" 0.198" y=" 0.198"/>
-  <xacro:quad_rotor name="rl" x="-0.198" y=" 0.198"/>
-  <xacro:quad_rotor name="rr" x="-0.198" y="-0.198"/>
-  <!-- Base link: central hub (inertia and collision unchanged for physics) -->
+  <!-- Stereo camera housing (ZED 2 class: 175 mm wide for a 120 mm baseline) -->
+  <xacro:property name="camera_width" value="0.175"/>
+  <xacro:property name="camera_height" value="0.03"/>
+  <xacro:property name="camera_depth" value="0.033"/>
+  <xacro:property name="motor_offset" value="0.174"/>
+  <!-- Upstream x500 props are 13" meshes scaled to 11" -->
+  <xacro:property name="prop_scale" value="0.8461538461538461"/>
+  <!-- Base link: frame mesh (inertia and main collision unchanged for physics) -->
   <link name="base_link">
     <inertial>
@@ -77,11 +26,8 @@
     </inertial>
     <visual>
-      <!-- Small central hub — arms provide the full quad silhouette -->
-      <geometry>
-        <box size="0.18 0.18 0.06"/>
-      </geometry>
-      <material name="body_dark">
-        <color rgba="0.12 0.12 0.12 1"/>
-      </material>
+      <origin xyz="0 0 0.025" rpy="0 0 ${pi}"/>
+      <geometry>
+        <mesh filename="${mesh_dir}/x500_frame.dae"/>
+      </geometry>
     </visual>
     <collision>
@@ -91,5 +37,90 @@
       </geometry>
     </collision>
+    <!-- Landing gear: two inclined legs and two skids (from the x500 model) -->
+    <collision>
+      <origin xyz="0 -0.098 -0.123" rpy="-0.35 0 0"/>
+      <geometry>
+        <box size="0.015 0.015 0.21"/>
+      </geometry>
+    </collision>
+    <collision>
+      <origin xyz="0 0.098 -0.123" rpy="0.35 0 0"/>
+      <geometry>
+        <box size="0.015 0.015 0.21"/>
+      </geometry>
+    </collision>
+    <collision>
+      <origin xyz="0 -0.132 -0.2195" rpy="0 0 0"/>
+      <geometry>
+        <box size="0.25 0.015 0.015"/>
+      </geometry>
+    </collision>
+    <collision>
+      <origin xyz="0 0.132 -0.2195" rpy="0 0 0"/>
+      <geometry>
+        <box size="0.25 0.015 0.015"/>
+      </geometry>
+    </collision>
   </link>
+  <!--
+    Motor + propeller macro (X configuration). The motor stator is a visual of
+    the rotor link, the propeller its own link so Gazebo can colour it.
+    Visuals stay unnamed: Gazebo Classic only applies <gazebo reference>
+    materials to visuals lumped through fixed joints when they keep their
+    default names.
+    Rotors are fixed: the drone is moved kinematically, see IMPLEMENTATION_PLAN.md.
+  -->
+  <xacro:macro name="quad_rotor" params="name x y prop">
+    <link name="rotor_${name}">
+      <inertial>
+        <!-- 4 x 0.035 kg keeps the total mass of the previous model -->
+        <mass value="0.035"/>
+        <inertia ixx="1e-5" ixy="0" ixz="0" iyy="1e-5" iyz="0" izz="1e-5"/>
+      </inertial>
+      <visual>
+        <origin xyz="0 0 -0.028" rpy="0 0 -0.45"/>
+        <geometry>
+          <mesh filename="${mesh_dir}/5010Base.dae"/>
+        </geometry>
+      </visual>
+      <visual>
+        <origin xyz="0 0 -0.032" rpy="0 0 0"/>
+        <geometry>
+          <mesh filename="${mesh_dir}/5010Bell.dae"/>
+        </geometry>
+      </visual>
+    </link>
+    <joint name="rotor_${name}_joint" type="fixed">
+      <parent link="base_link"/>
+      <child link="rotor_${name}"/>
+      <origin xyz="${x} ${y} 0.06" rpy="0 0 0"/>
+    </joint>
+    <link name="prop_${name}">
+      <visual>
+        <!-- The prop mesh origin is at its tip, this centres the hub on the motor -->
+        <origin xyz="-0.022 -0.14638461538461536 -0.016" rpy="0 0 0"/>
+        <geometry>
+          <mesh filename="${mesh_dir}/1345_prop_${prop}.stl"
+            scale="${prop_scale} ${prop_scale} ${prop_scale}"/>
+        </geometry>
+        <material name="prop_dark_grey">
+          <color rgba="0.175 0.175 0.175 1"/>
+        </material>
+      </visual>
+    </link>
+    <joint name="prop_${name}_joint" type="fixed">
+      <parent link="rotor_${name}"/>
+      <child link="prop_${name}"/>
+      <origin xyz="0 0 0" rpy="0 0 0"/>
+    </joint>
+    <gazebo reference="prop_${name}">
+      <material>Gazebo/DarkGrey</material>
+    </gazebo>
+  </xacro:macro>
+  <!-- PX4 quad-X numbering: FR and RL spin CCW, FL and RR spin CW -->
+  <xacro:quad_rotor name="fr" x="${motor_offset}" y="${-motor_offset}" prop="ccw"/>
+  <xacro:quad_rotor name="fl" x="${motor_offset}" y="${motor_offset}" prop="cw"/>
+  <xacro:quad_rotor name="rl" x="${-motor_offset}" y="${motor_offset}" prop="ccw"/>
+  <xacro:quad_rotor name="rr" x="${-motor_offset}" y="${-motor_offset}" prop="cw"/>
   <!-- IMU link -->
   <link name="imu_link">
@@ -104,5 +135,8 @@
     <origin xyz="0 0 0"/>
   </joint>
-  <!-- Stereo camera mount link -->
+  <!--
+    Stereo camera mount link: housing hung from the front of the payload rails
+    (underside z = -0.026, front end x = 0.15), below the propeller discs.
+  -->
   <link name="stereo_camera_link">
     <inertial>
@@ -112,5 +146,5 @@
     <visual>
       <geometry>
-        <box size="${camera_width} ${camera_height} ${camera_depth}"/>
+        <box size="${camera_depth} ${camera_width} ${camera_height}"/>
       </geometry>
       <material name="dark_gray">
@@ -118,15 +152,52 @@
       </material>
     </visual>
-    <collision>
-      <geometry>
-        <box size="${camera_width} ${camera_height} ${camera_depth}"/>
+    <visual>
+      <!-- Bracket plate between the rails and the housing -->
+      <origin xyz="-0.0375 0 0.0135" rpy="0 0 0"/>
+      <geometry>
+        <box size="0.085 0.05 0.003"/>
+      </geometry>
+      <material name="dark_gray">
+        <color rgba="0.2 0.2 0.2 1"/>
+      </material>
+    </visual>
+    <collision>
+      <geometry>
+        <box size="${camera_depth} ${camera_width} ${camera_height}"/>
       </geometry>
     </collision>
   </link>
+  <gazebo reference="stereo_camera_link">
+    <material>Gazebo/DarkGrey</material>
+  </gazebo>
+  <!-- Lens macro: glass disc on the front face, in front of each camera frame -->
+  <xacro:macro name="stereo_lens" params="side">
+    <link name="stereo_${side}_lens_link">
+      <visual>
+        <origin xyz="0 0 0" rpy="0 ${pi/2} 0"/>
+        <geometry>
+          <cylinder radius="0.009" length="0.004"/>
+        </geometry>
+        <material name="lens_black">
+          <color rgba="0.02 0.02 0.03 1"/>
+        </material>
+      </visual>
+    </link>
+    <joint name="stereo_${side}_lens_joint" type="fixed">
+      <parent link="stereo_${side}_camera_frame"/>
+      <child link="stereo_${side}_lens_link"/>
+      <origin xyz="${camera_depth/2} 0 0" rpy="0 0 0"/>
+    </joint>
+    <gazebo reference="stereo_${side}_lens_link">
+      <material>Gazebo/Black</material>
+    </gazebo>
+  </xacro:macro>
+  <xacro:stereo_lens side="left"/>
+  <xacro:stereo_lens side="right"/>
   <!-- Camera mount joint -->
   <joint name="camera_mount_joint" type="fixed">
     <parent link="base_link"/>
     <child link="stereo_camera_link"/>
-    <origin xyz="0.2 0 0.05" rpy="0 0 0"/>
+    <origin xyz="0.2 0 -0.0375" rpy="0 0 0"/>
   </joint>
   <!-- Left camera optical frame -->
@@ -158,8 +229,5 @@
     <origin xyz="0 0 0" rpy="${-pi/2} 0 ${-pi/2}"/>
   </joint>
-  <!-- Gazebo plugins -->
-  <gazebo reference="base_link">
-    <material>Gazebo/Black</material>
-  </gazebo>
+  <!-- Gazebo plugins (base_link has no material override: the frame mesh carries its own) -->
   <!-- Left camera sensor -->
   <gazebo reference="stereo_left_camera_frame">

Commit message: Run YOLO on the GPU when available and silence gzclient model warnings
- target_detector: new default device 'auto' picks cuda:0 when PyTorch
  sees a GPU and falls back to the CPU otherwise, logging why. The
  perception launch file no longer hardcodes 'cpu'.
- URDF: reference meshes with file://$(find interceptor_drone) instead of
  package://, and drop the gazebo_model_path export that put the install
  share/ directory on GAZEBO_MODEL_PATH. gzclient's Insert tab scanned
  that directory and logged "Missing model.config" for every package in it.

Co-Authored-By: Claude Opus 5.5 <noreply@anthropic.com>
Claude-Session: https://claude.ai/code/session_01FqLzMcYSgygF4F38WJEpKJ

File: interceptor_ws/src/interceptor_drone/urdf/interceptor_quadrotor.urdf.xacro (robot description, xacro)
@@ -9,5 +9,10 @@
   -->
   <!-- Property definitions -->
-  <xacro:property name="mesh_dir" value="package://interceptor_drone/meshes/x500"/>
+  <!--
+    Absolute file:// URIs work in both Gazebo and RViz without adding the
+    install share/ directory to GAZEBO_MODEL_PATH (which makes gzclient's
+    Insert tab log "Missing model.config" for every package in it).
+  -->
+  <xacro:property name="mesh_dir" value="file://$(find interceptor_drone)/meshes/x500"/>
   <xacro:property name="camera_mass" value="0.1"/>
   <xacro:property name="baseline" value="0.12"/>

Commit message: Add quadrotor flight dynamics, flight controller and keyboard teleop
The drone can now fly in Gazebo on a physics model instead of being a
static model:

- Flight dynamics library (interceptor_drone_flight, plain C++/Eigen):
  first-order motor lag, rotor thrust T = k_f w^2 with reaction torque
  Q = k_m T, rotor (blade-flapping) drag, quadratic airframe drag on the
  airspeed, rotational damping, Cheeseman-Bennett ground effect, air
  density scaling, and steady wind with Gauss-Markov gusts. Rotor
  coefficients are the PX4 x500 SITL values.
- Onboard flight controller: velocity PI -> thrust vector with tilt
  limit -> geometric attitude P -> body-rate PI -> mixer with roll/pitch
  priority on saturation, plus a landed/take-off state.
- quadrotor_dynamics Gazebo plugin: runs controller and plant every
  physics step, applies the wrench to base_link, spins the propellers,
  publishes /odom, TF odom->base_link, /joint_states, /drone/status and
  /drone/wind. Inputs: /cmd_vel, /drone/arm, /drone/set_wind.
- drone_teleop_keyboard.py: arrow keys / WASD teleop node (make teleop).
- URDF: propellers on continuous joints, plugin block; wind set via
  simulation.launch.py args. The drone spawns at (-3, -3), off the walking
  person's patrol path in the existing park world.
- 22 gtests, including closed-loop hover, velocity, yaw, wind rejection
  and take-off/touchdown in a standalone 6-DOF sim.
- docs/FLIGHT_DYNAMICS.md; README, CLAUDE.md and the plan updated.

Co-Authored-By: Claude Opus 5.5 <noreply@anthropic.com>
Claude-Session: https://claude.ai/code/session_013kzc7cphvXaVk47PELexQy

File: interceptor_ws/src/interceptor_drone/urdf/interceptor_quadrotor.urdf.xacro (robot description, xacro)
@@ -7,5 +7,13 @@
     unchanged. Landing-gear collisions let the drone rest on its skids, and the
     stereo camera hangs under the payload rails so it clears the propellers.
+    Flight: the quadrotor_dynamics plugin at the end of this file computes rotor
+    thrust, reaction torques, aerodynamic drag, wind and ground effect, and runs
+    the onboard flight controller (see src/flight/ and docs/FLIGHT_DYNAMICS.md).
   -->
+  <!-- Wind (world frame, m/s), set from simulation.launch.py -->
+  <xacro:arg name="wind_x" default="0.0"/>
+  <xacro:arg name="wind_y" default="0.0"/>
+  <xacro:arg name="wind_z" default="0.0"/>
+  <xacro:arg name="wind_gust_stddev" default="0.0"/>
   <!-- Property definitions -->
   <xacro:property name="mesh_dir" value="package://interceptor_drone/meshes/x500"/>
@@ -69,11 +77,12 @@
     materials to visuals lumped through fixed joints when they keep their
     default names.
-    Rotors are fixed: the drone is moved kinematically, see IMPLEMENTATION_PLAN.md.
+    The propeller spins on a continuous joint. Its speed is set by the dynamics
+    plugin (visual only, slowed down); thrust is applied to base_link.
   -->
   <xacro:macro name="quad_rotor" params="name x y prop">
     <link name="rotor_${name}">
       <inertial>
-        <!-- 4 x 0.035 kg keeps the total mass of the previous model -->
-        <mass value="0.035"/>
+        <!-- Motor 0.030 kg + propeller 0.005 kg keeps the total mass of the previous model -->
+        <mass value="0.030"/>
         <inertia ixx="1e-5" ixy="0" ixz="0" iyy="1e-5" iyz="0" izz="1e-5"/>
       </inertial>
@@ -97,4 +106,8 @@
     </joint>
     <link name="prop_${name}">
+      <inertial>
+        <mass value="0.005"/>
+        <inertia ixx="1e-6" ixy="0" ixz="0" iyy="3.3e-5" iyz="0" izz="3.3e-5"/>
+      </inertial>
       <visual>
         <!-- The prop mesh origin is at its tip, this centres the hub on the motor -->
@@ -109,8 +122,9 @@
       </visual>
     </link>
-    <joint name="prop_${name}_joint" type="fixed">
+    <joint name="prop_${name}_joint" type="continuous">
       <parent link="rotor_${name}"/>
       <child link="prop_${name}"/>
       <origin xyz="0 0 0" rpy="0 0 0"/>
+      <axis xyz="0 0 1"/>
     </joint>
     <gazebo reference="prop_${name}">
@@ -313,3 +327,52 @@
     </sensor>
   </gazebo>
+  <!--
+    Flight dynamics + onboard flight controller.
+    Rotor coefficients are the PX4 x500 SITL values. Mass and inertia are read
+    from this model, rotor positions from the prop joints.
+    Topics: cmd_vel (in), drone/arm (in), drone/set_wind (in), odom, joint_states,
+    drone/status, drone/wind (out), TF odom -> base_link.
+  -->
+  <gazebo>
+    <plugin name="quadrotor_dynamics" filename="libquadrotor_dynamics_plugin.so">
+      <ros>
+        <namespace>/</namespace>
+      </ros>
+      <body_link>base_link</body_link>
+      <rotor><joint>prop_fr_joint</joint><direction>ccw</direction></rotor>
+      <rotor><joint>prop_fl_joint</joint><direction>cw</direction></rotor>
+      <rotor><joint>prop_rl_joint</joint><direction>ccw</direction></rotor>
+      <rotor><joint>prop_rr_joint</joint><direction>cw</direction></rotor>
+      <!-- Rotors: T = k_f w^2, Q = k_m T, first-order motor lag -->
+      <thrust_coefficient>8.54858e-06</thrust_coefficient>
+      <moment_coefficient>0.016</moment_coefficient>
+      <rotor_drag_coefficient>8.06428e-05</rotor_drag_coefficient>
+      <rotor_radius>0.1397</rotor_radius>
+      <max_rotor_speed>1000.0</max_rotor_speed>
+      <motor_time_constant_up>0.0125</motor_time_constant_up>
+      <motor_time_constant_down>0.025</motor_time_constant_down>
+      <rotor_visual_slowdown>10.0</rotor_visual_slowdown>
+      <!-- Aerodynamics -->
+      <air_density>1.225</air_density>
+      <drag_area>0.04 0.04 0.08</drag_area>
+      <angular_drag>0.002</angular_drag>
+      <ground_effect>true</ground_effect>
+      <ground_height>0.0</ground_height>
+      <wind_mean>$(arg wind_x) $(arg wind_y) $(arg wind_z)</wind_mean>
+      <wind_gust_stddev>$(arg wind_gust_stddev)</wind_gust_stddev>
+      <wind_gust_time_constant>2.0</wind_gust_time_constant>
+      <!-- Flight controller -->
+      <command_frame>heading</command_frame>
+      <command_timeout>0.5</command_timeout>
+      <max_horizontal_speed>8.0</max_horizontal_speed>
+      <max_vertical_speed>3.0</max_vertical_speed>
+      <max_yaw_rate>1.5</max_yaw_rate>
+      <max_tilt>0.61</max_tilt>
+      <idle_rotor_speed>100.0</idle_rotor_speed>
+      <start_armed>false</start_armed>
+      <odom_frame>odom</odom_frame>
+      <odom_rate>100.0</odom_rate>
+      <joint_state_rate>30.0</joint_state_rate>
+    </plugin>
+  </gazebo>
 </robot>

Commit message: feat(perception): Make the vision path work and add the bicycle class (P2.5)
The vision pipeline never produced a usable detection. Four separate
problems had to be fixed.

1. The detector died at import. The ROS 2 Humble cv_bridge Python binding
   is compiled against the NumPy 1.x C API, so with the NumPy 2 of the
   image "import cv_bridge" raises "AttributeError: _ARRAY_API not found"
   and then segfaults. target_detector.py decodes the sensor_msgs/Image
   with NumPy instead, which works with NumPy 1 and 2 alike. The Dockerfile
   pins numpy<2 as well, so a rebuilt image gets the binding back.

2. The stereo pair was mirrored. The URDF put the camera called "left" at
   -baseline/2 in a FLU body frame, so it was physically the right one and
   the disparity of the pair was negative. SGBM (minDisparity 0) cannot
   match a negative disparity, so the depth of the whole scene was the sky.
   The two joint origins are swapped now.

3. SGBM with 128 disparities dropped the target's disparity completely.
   With 64 the person's box is 100 % valid with a disparity of 7.9 px at
   8.4 m, and the depth image went from 12 % to 90 % valid pixels.

4. The depth processor's focal length was 535.4 instead of the camera's
   554.38 (from the URDF's 640 px width and 1.047 rad field of view).

The detector also reports the COCO bicycle (class 1) as
TargetDetection.BICYCLE now, and the class list is a parameter so the
detector and the tracker's follow.eligible_classes agree on the names and
ids. The device selection is explicit and logged: which device was picked
and why it fell back to the CPU.

The Dockerfile pins torch 2.6.0 / torchvision 0.21.0, the CUDA 12.4 build.
The torch 2.14.1+cu130 of the image asks for a newer driver than the host
has (555.97, i.e. CUDA 12.5), so torch.cuda.is_available() stayed False
and the detector silently ran on the CPU. The image has to be rebuilt for
the pin to take effect.

Verified in Gazebo with the walker as the target: YOLO detects the person
at 0.6-0.9 confidence, the localizer turns the detections into 3D
positions with a median 0.36 m horizontal error against the ground truth,
and the tracker confirms the track (100 % of the track samples on the GPU).

Co-Authored-By: Claude Code <noreply@anthropic.com>

File: interceptor_ws/src/interceptor_drone/urdf/interceptor_quadrotor.urdf.xacro (robot description, xacro)
@@ -223,9 +223,16 @@
   </joint>
   <!-- Left camera optical frame -->
+  <!--
+    The body frame is FLU (x forward, y left, z up), so the LEFT camera sits at
+    +baseline/2 in y and the RIGHT camera at -baseline/2. The other way round the
+    two images are mirrored: the object appears further left in the image of the
+    camera on the right, so the disparity of the pair is negative and the SGBM
+    matcher (minDisparity 0) cannot find it. The depth came out as the sky.
+  -->
   <link name="stereo_left_camera_frame"/>
   <joint name="stereo_left_camera_joint" type="fixed">
     <parent link="stereo_camera_link"/>
     <child link="stereo_left_camera_frame"/>
-    <origin xyz="0 ${-baseline/2} 0" rpy="0 0 0"/>
+    <origin xyz="0 ${baseline/2} 0" rpy="0 0 0"/>
   </joint>
   <!-- Right camera optical frame -->
@@ -234,5 +241,5 @@
     <parent link="stereo_camera_link"/>
     <child link="stereo_right_camera_frame"/>
-    <origin xyz="0 ${baseline/2} 0" rpy="0 0 0"/>
+    <origin xyz="0 ${-baseline/2} 0" rpy="0 0 0"/>
   </joint>
   <!-- Left camera optical link (ROS convention: Z forward, X right, Y down) -->
